File: Bussystem/Bussystem.kicad_pcb (KiCad board)
At the start: 2 copper layers, 100 x 60 mm, 11 parts, among them J1 PCIE-098-02-X-D-TH, J2 PCIE-098-02-X-D-TH, J3 PCIE-098-02-X-D-TH, J4 PCIE-098-02-X-D-TH, J5 PCIE-098-02-X-D-TH, J6 PCIE-098-02-X-D-EMS2-BG, J7 8x Edge conn

Commit message: first 10x Bus baseplate design. Still needs some redesign
Parts:
- moved H1 24.1 mm to (135.0, 119.0)
- moved H3 21.1 mm to (135.0, 94.0)
- moved H6 5.00 mm to (58.0, 119.0)
- moved H4 3.16 mm to (58.0, 94.0)
- moved J2 3.00 mm to (81.8, 105.0)
- moved J3 3.00 mm to (96.8, 105.0)
- moved J4 3.00 mm to (111.8, 105.0)
- moved J5 3.00 mm to (126.8, 105.0)
- moved J1 3.00 mm to (66.8, 105.0)
