File: Bussystem/Bussystem 10x non stack.sch (KiCad schematic (older format))
At the start: 13 parts, among them J1 PCIE-098-02-X-D-TH, J10 PCIE-098-02-X-D-TH, J2 PCIE-098-02-X-D-TH, J3 PCIE-098-02-X-D-TH, J4 PCIE-098-02-X-D-TH, J5 PCIE-098-02-X-D-TH, J6 PCIE-098-02-X-D-TH, J7 PCIE-098-02-X-D-TH, J8 PCIE-098-02-X-D-TH, J9 PCIE-098-02-X-D-TH

Commit message: some new parts in the Buscontroller T1
Parts:
- J1, J10, J2, J3, J4, J5, J6, J7, J8, J9: symbol PCIE-098-02-X-D-TH:PCIE-098-02-X-D-TH -> Bussystem-10x-non-stack-rescue:PCIE-098-02-X-D-TH-PCIE-098-02-X-D-TH
Changed lines of the file:
@@
 $EndDescr
 $Comp
-L PCIE-098-02-X-D-TH:PCIE-098-02-X-D-TH J1
+L Bussystem-10x-non-stack-rescue:PCIE-098-02-X-D-TH-PCIE-098-02-X-D-TH J1
 U 1 1 60CF1FEA
 P 2050 3450
@@
 $EndComp
 $Comp
-L PCIE-098-02-X-D-TH:PCIE-098-02-X-D-TH J2
+L Bussystem-10x-non-stack-rescue:PCIE-098-02-X-D-TH-PCIE-098-02-X-D-TH J2
 U 1 1 60CF3AF9
 P 3350 3450
@@
 	2850 5850 2550 5850
 $Comp
-L PCIE-098-02-X-D-TH:PCIE-098-02-X-D-TH J3
+L Bussystem-10x-non-stack-rescue:PCIE-098-02-X-D-TH-PCIE-098-02-X-D-TH J3
 U 1 1 60D17DD6
 P 4650 3450
@@
 	4150 5850 3850 5850
 $Comp
-L PCIE-098-02-X-D-TH:PCIE-098-02-X-D-TH J4
+L Bussystem-10x-non-stack-rescue:PCIE-098-02-X-D-TH-PCIE-098-02-X-D-TH J4
 U 1 1 60D29B40
 P 5950 3450
@@
 	5450 5850 5150 5850
 $Comp
-L PCIE-098-02-X-D-TH:PCIE-098-02-X-D-TH J5
+L Bussystem-10x-non-stack-rescue:PCIE-098-02-X-D-TH-PCIE-098-02-X-D-TH J5
 U 1 1 60D29B7F
 P 7250 3450
@@
 	5300 1100 6600 1100
 $Comp
-L PCIE-098-02-X-D-TH:PCIE-098-02-X-D-TH J6
+L Bussystem-10x-non-stack-rescue:PCIE-098-02-X-D-TH-PCIE-098-02-X-D-TH J6
 U 1 1 61072508
 P 8550 3450
@@
 Connection ~ 6600 2100
 $Comp
-L PCIE-098-02-X-D-TH:PCIE-098-02-X-D-TH J7
+L Bussystem-10x-non-stack-rescue:PCIE-098-02-X-D-TH-PCIE-098-02-X-D-TH J7
 U 1 1 610F5708
 P 9850 3450
@@
 	9350 5850 9050 5850
 $Comp
-L PCIE-098-02-X-D-TH:PCIE-098-02-X-D-TH J8
+L Bussystem-10x-non-stack-rescue:PCIE-098-02-X-D-TH-PCIE-098-02-X-D-TH J8
 U 1 1 610F5747
 P 11150 3450
@@
 	10650 5850 10350 5850
 $Comp
-L PCIE-098-02-X-D-TH:PCIE-098-02-X-D-TH J9
+L Bussystem-10x-non-stack-rescue:PCIE-098-02-X-D-TH-PCIE-098-02-X-D-TH J9
 U 1 1 610F5786
 P 12450 3450
@@
 	10500 1100 11800 1100
 $Comp
-L PCIE-098-02-X-D-TH:PCIE-098-02-X-D-TH J10
+L Bussystem-10x-non-stack-rescue:PCIE-098-02-X-D-TH-PCIE-098-02-X-D-TH J10
 U 1 1 610F585F
 P 13750 3450
